File: HSTC/HSTC.kicad_sch (KiCad schematic)
At the start: 119 parts, among them IC1 PIC16C620A-04/SS, IC2 PIC16C620A-04/SS, J1 Conn_01x05_Pin, J2 Conn_01x05_Pin, J3 Conn_01x04_Pin, J4 Conn_01x04_Pin, J5 Conn_01x04_Pin, J7 Conn_01x05_Pin, Q1 BCX56, Q10 IMX1T110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

Commit message: Add files via upload
14/10/25
Connections:
- net at C9.2, J1.2 (Pin_2), Q1.2 (C)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: no longer C1.1, J1.4 (Pin_4)
- net at Q12.2 (C), R42.1: now also C1.1, J1.4 (Pin_4)
Other:
- note added: "Checked"
- moved on the sheet: C1
